File: wroom02_alarm.sch (KiCad schematic (older format))
At the start: 7 parts

Commit message: 基本回路
Parts:
- added Q1: Q_NMOS_GDS, symbol Q_NMOS_GDS
- added R6: 100, symbol R
- added R7: 10k, symbol R
- added SW1: Write, symbol switch
- added SW2: RESET, symbol switch
- J1: renamed from J?; value CONN_01X03 -> Serial
- gave numbers to parts that had none: 6
Connections:
- wire segments 29 -> 34
Other:
- moved on the sheet: J1, R5

Commit message: DRCエラーを修正
Parts:
- added C1, C2: 0.1u, symbol C
- added C3: CP, symbol CP
- added D1: LED, symbol LED
- added J10, J11, J4, J5, J6, J7, J8, J9: pin, symbol CONN_01X01
- added J2: BARREL_JACK, symbol BARREL_JACK
- added J3: microUSB, symbol microUSB
- added R8: 1k, symbol R
- added RL1: Y14H-1C-5DS, symbol Y14H-1C-5DS
- added U3: 7803, symbol 7805
Connections:
- net +3V3: now also C2.1, C3.1, U3.VO
- net GND: now also C1.2, C2.2, C3.2, D1.1 (K), J2.2, J2.3, J3.5 (GND), U3.GND
- net at U1.10 (IO4): now also J11.1 (P1)
- net at U1.14 (IO5): now also J10.1 (P1)
- net at U1.16 (TOUT): now also J9.1 (P1)
- net at U1.3 (IO14): now also J6.1 (P1)
- net at U1.4 (IO12): now also J7.1 (P1)
- net at U1.5 (IO13): now also J8.1 (P1)
- net at Q1.2 (D): now also RL1.2
- new net: D1.2 (A), R8.2
- new net: J3.2 (D-), J4.1 (P1)
- new net: J3.3 (D+), J5.1 (P1)
- new net +5V: C1.1, J2.1, J3.1 (VBAS), R8.1, RL1.5, U3.VI
- no-connect marks 0 -> 1

Commit message: 基板も完成
Parts:
- removed J2: BARREL_JACK, symbol BARREL_JACK
- added J12, J13, J14, J15, J2: pin, pad:universal, symbol CONN_01X01
- C1, C2: footprint (none) -> Capacitors_SMD:C_0603_HandSoldering
- C3: footprint (none) -> Capacitors_THT:CP_Radial_D8.0mm_P2.50mm
- D1: footprint (none) -> LEDs:LED_0603_HandSoldering
- J1: footprint (none) -> Pin_Headers:Pin_Header_Straight_1x03_Pitch2.54mm
- J10, J11, J4, J5, J6, J7, J8, J9: footprint (none) -> pad:universal
- J3: footprint (none) -> lib:microUSB
- Q1: footprint (none) -> TO_SOT_Packages_THT:TO-220_Vertical
- R1, R2, R3, R4, R5, R6, R7, R8: footprint (none) -> Resistors_SMD:R_0603_HandSoldering
- RL1: footprint (none) -> lib:Y14H-1C-5DS
- SW1, SW2: footprint (none) -> lib:switch
- U1: footprint (none) -> lib:WROOM02
- U3: footprint (none) -> TO_SOT_Packages_SMD:TO-252-3_TabPin2
Connections:
- net +3V3: now also J14.1 (P1)
- net GND: now also J15.1 (P1)
- net at RL1.1: now also J13.1 (P1)
- net at RL1.3 (NO): now also J12.1 (P1)
- net at RL1.4 (NC): now also J2.1 (P1)
- no-connect marks 1 -> 2
Other:
- moved on the sheet: J3, J4, J5, Q1, R6, R7, RL1

Commit message: GBRを作成
Parts:
- removed J12, J13: pin, pad:universal, symbol CONN_01X01
- added D?: LED, symbol LED
- Q1: value Q_NMOS_GDS -> 2SK4017
Connections:
- net GND: now also RL1.1
- net at RL1.3 (NO): now also D?.1 (K)
- new net +12V: D?.2 (A)
Changed lines of the file:
@@
 P 8300 3250
 F 0 "Q1" H 8500 3300 50  0000 L CNN
-F 1 "Q_NMOS_GDS" H 8500 3200 50  0000 L CNN
+F 1 "2SK4017" H 8500 3200 50  0000 L CNN
 F 2 "TO_SOT_Packages_THT:TO-220_Vertical" H 8500 3350 50  0001 C CNN
 F 3 "" H 8300 3250 50  0001 C CNN
@@
 Connection ~ 4950 1000
 $Comp
-L CONN_01X01 J12
-U 1 1 5977493D
-P 8200 2200
-F 0 "J12" H 8300 2200 50  0000 C CNN
-F 1 "pin" V 8300 2200 50  0001 C CNN
-F 2 "pad:universal" H 8200 2200 50  0001 C CNN
-F 3 "" H 8200 2200 50  0001 C CNN
-	1    8200 2200
-	1    0    0    -1
-$EndComp
-$Comp
-L CONN_01X01 J13
-U 1 1 59774AC7
-P 8200 2650
-F 0 "J13" H 8300 2650 50  0000 C CNN
-F 1 "pin" V 8300 2650 50  0001 C CNN
-F 2 "pad:universal" H 8200 2650 50  0001 C CNN
-F 3 "" H 8200 2650 50  0001 C CNN
-	1    8200 2650
-	1    0    0    -1
-$EndComp
-$Comp
 L CONN_01X01 J2
 U 1 1 59774BA2
@@
 Wire Wire Line
 	6600 1350 6650 1350
+$Comp
+L +12V #PWR?
+U 1 1 597A254A
+P 10000 1650
+F 0 "#PWR?" H 10000 1500 50  0001 C CNN
+F 1 "+12V" H 10000 1790 50  0000 C CNN
+F 2 "" H 10000 1650 50  0001 C CNN
+F 3 "" H 10000 1650 50  0001 C CNN
+	1    10000 1650
+	1    0    0    -1
+$EndComp
+$Comp
+L LED D?
+U 1 1 597A25A0
+P 10000 1950
+F 0 "D?" H 10000 2050 50  0000 C CNN
+F 1 "LED" H 10000 1850 50  0000 C CNN
+F 2 "" H 10000 1950 50  0001 C CNN
+F 3 "" H 10000 1950 50  0001 C CNN
+	1    10000 1950
+	0    -1   -1   0
+$EndComp
+$Comp
+L GND #PWR?
+U 1 1 597A262D
+P 9950 2750
+F 0 "#PWR?" H 9950 2500 50  0001 C CNN
+F 1 "GND" H 9950 2600 50  0000 C CNN
+F 2 "" H 9950 2750 50  0001 C CNN
+F 3 "" H 9950 2750 50  0001 C CNN
+	1    9950 2750
+	1    0    0    -1
+$EndComp
+Wire Wire Line
+	10000 1650 10000 1800
+Wire Wire Line
+	8000 2200 10000 2200
+Wire Wire Line
+	10000 2200 10000 2100
+Wire Wire Line
+	9950 2650 8000 2650
+Wire Wire Line
+	9950 2650 9950 2750
 $EndSCHEMATC
